File: ziptie-keyboard-v0.2.kicad_pcb (KiCad board)
At the start: 2 copper layers, 29.3 x 11.3 mm, 147 parts, among them SW1 RotaryEncoder, U1 nice_nano

Commit message: Updated traces to 1mm and traced matrix
Parts:
- moved U1 8.41 mm to (31.8, 22.5)
Connections:
- U1 pad 1: COL-5 -> COL-0
- U1 pad 10: ROW-1 -> COL-7
- U1 pad 11: ROW-2 -> COL-8
- U1 pad 12: ROW-3 -> COL-9
- U1 pad 14: COL-12 -> ROW-4
- U1 pad 15: COL-11 -> ROW-3
- U1 pad 16: COL-10 -> ROW-2
- U1 pad 17: COL-9 -> ROW-1
- U1 pad 18: COL-8 -> ROW-0
- U1 pad 19: COL-7 -> ROT-B
- U1 pad 2: COL-4 -> COL-1
- U1 pad 20: COL-6 -> ROT-A
- U1 pad 23: unconnected-(U1-GND-Pad23) -> ROT-GRD
- U1 pad 3: ROT-GRD -> unconnected-(U1-GND-Pad3)
- U1 pad 31: ROW-4 -> COL-10
- U1 pad 32: ROT-B -> COL-11
- U1 pad 33: ROT-A -> COL-12
- U1 pad 5: COL-3 -> COL-2
- U1 pad 6: COL-2 -> COL-3
- U1 pad 7: COL-1 -> COL-4
- U1 pad 8: COL-0 -> COL-5
- U1 pad 9: ROW-0 -> COL-6
Routing:
- net ROW-4: track 0.00 -> 331.3 mm
- net ROW-3: track 0.00 -> 307.5 mm
- net ROW-2: track 0.00 -> 305.0 mm
- net ROW-0: track 0.00 -> 258.7 mm
- net ROW-1: track 0.00 -> 257.2 mm
- net COL-10: track 0.00 -> 116.3 mm
- net COL-12: track 0.00 -> 114.7 mm
- net COL-11: track 0.00 -> 112.2 mm
- net COL-9: track 0.00 -> 107.2 mm
- net COL-8: track 0.00 -> 104.8 mm
- net COL-6: track 0.00 -> 104.8 mm
- net COL-7: track 0.00 -> 104.8 mm
- net COL-5: track 0.00 -> 99.0 mm
- net COL-13: track 0.00 -> 95.3 mm
- net COL-1: track 0.00 -> 93.0 mm
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
Commit message: Added traces and board cuts
Parts:
- added J1: Conn_01x01_Socket, Connector_Wire:SolderWire-0.1sqmm_1x01_D0.4mm_OD1mm, F.Cu at (220.7, 37.3)
- added J2: Conn_01x01_Socket, Connector_Wire:SolderWire-0.1sqmm_1x01_D0.4mm_OD1mm, F.Cu at (218.3, 31.8)
- moved U1 7.66 mm to (31.0, 30.2)
Connections:
- U1 pad 13: COL-13 -> ROT-A
- U1 pad 14: ROW-4 -> ROW-0
- U1 pad 15: ROW-3 -> ROW-1
- U1 pad 17: ROW-1 -> ROW-3
- U1 pad 18: ROW-0 -> ROW-4
- U1 pad 20: ROT-A -> COL-13
- U1 pad 21: unconnected-(U1-VCC-Pad21) -> PWR VCC
- U1 pad 3: unconnected-(U1-GND-Pad3) -> PWR GRD
Routing:
- net ROT-GRD: track 0.00 -> 310.2 mm
- net ROT-B: track 0.00 -> 294.0 mm
- net ROT-A: track 0.00 -> 280.9 mm
- net COL-13: track 95.3 -> 356.6 mm
- net PWR GRD: track 0.00 -> 228.3 mm
- net COL-12: track 114.7 -> 331.5 mm
- net PWR VCC: track 0.00 -> 203.5 mm
- net COL-11: track 112.2 -> 309.4 mm
- net COL-10: track 116.3 -> 293.0 mm
- net COL-9: track 107.2 -> 258.8 mm
- net COL-8: track 104.8 -> 241.6 mm
- net ROW-4: track 331.3 -> 466.5 mm
- net ROW-3: track 307.5 -> 430.9 mm
- net COL-7: track 104.8 -> 225.0 mm
- net ROW-2: track 305.0 -> 422.7 mm
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Other:
- board size 29.3 x 11.3 mm -> 322.3 x 125.4 mm
